Commit message: feat: URDF робота изменен для Gazebo

File: agrolab_description/urdf/agrolab.urdf (robot description, URDF)
Before this commit: robot agrolab, 7 links, 6 joints
Joints:
- removed joint X_to_Y
- removed joint Y_to_Z
- removed joint base_link_to_X
- added joint ${base_link_to_x}: type prismatic, parent base_link, child X, axis 1 0 0, limit lower=0 upper=0.43 effort=10000 velocity=1
- added joint ${x_to_y}: type prismatic, parent X, child Y, axis 0 1 0, limit lower=0 upper=0.54 effort=10000 velocity=1
- added joint ${y_to_z}: type prismatic, parent Y, child Z, axis 0 0 -1, limit lower=0 upper=0.2 effort=10000 velocity=1

Commit message: added camera (not tested fix to arm)

File: agrolab_description/urdf/agrolab.urdf (robot description, URDF)
Before this commit: robot agrolab, 7 links, 6 joints
Links:
- added link camera_link; collision box size=0.01 0.01 0.01; visual box size=0.01 0.01 0.01
Joints:
- added joint camera_joint: type fixed, parent Y, child camera_link, origin xyz=-0.26 -0.26 0.4 rpy=0 1.57 0, axis 0 1 0

Commit message: added working with gazebo

File: agrolab_description/urdf/agrolab.urdf (robot description, URDF)
Before this commit: robot agrolab, 7 links, 6 joints
Links:
- added link Camera, mass 0.01; collision box size=0.02 0.02 0.02; visual box size=0.02 0.02 0.02
- added link gripper_link1, mass 0.01; collision mesh filename=package://agrolab_description/meshes/link7.dae scale=0.001 0.001 0.001; visual mesh filename=package://agrolab_description/meshes/link7.dae scale=0.001 0.001 0.001
- added link gripper_link2, mass 0.01; collision mesh filename=package://agrolab_description/meshes/link7.dae scale=0.001 0.001 0.001; visual mesh filename=package://agrolab_description/meshes/link7.dae scale=0.001 0.001 0.001
- link Water_tank: mass 0.5 -> 1.5
- link base_link: mass 7 -> 20
Joints:
- removed joint ${base_link_to_x}
- removed joint ${x_to_y}
- removed joint ${y_to_z}
- added joint Camera2Light: type fixed, parent Light, child Camera, origin xyz=0 0 0.7 rpy=0 1.57 0
- added joint X_to_Y: type prismatic, parent X, child Y, axis 0 1 0, limit lower=0 upper=0.54 effort=10000 velocity=1
- added joint Y_to_Z: type prismatic, parent Y, child Z, axis 0 0 -1, limit lower=0 upper=0.2 effort=10000 velocity=1
- added joint base_link_to_X: type prismatic, parent base_link, child X, axis 1 0 0, limit lower=0 upper=0.43 effort=10000 velocity=1
- added joint gripper: type prismatic, parent Z, child gripper_link1, origin xyz=-0.22 -0.26 0.25 rpy=1.57 3.14 0, axis 0 0 1, limit lower=0 upper=0.040 effort=3 velocity=0.05
- added joint gripper_sub: type prismatic, parent Z, child gripper_link2, origin xyz=-0.22 -0.26 0.25 rpy=-1.57 0 0, axis 0 0 1, limit lower=0 upper=0.040 effort=3 velocity=0.05

Commit message: added camera attached to Y_joint

File: agrolab_description/urdf/agrolab.urdf (robot description, URDF)
Before this commit: robot agrolab, 10 links, 9 joints
Joints:
- joint Camera2Light: origin xyz=0 0 0.7 rpy=0 1.57 0 -> xyz=-0.26 -0.26 0.4 rpy=0 1.57 0; parent Light -> Y; type fixed -> continuous

Commit message: added red sphere to urdf

File: agrolab_description/urdf/agrolab.urdf (robot description, URDF)
Before this commit: robot agrolab, 10 links, 9 joints
Links:
- added link sphere1; visual sphere radius=0.02
Joints:
- added joint sphere1: type fixed, parent base_link, child sphere1, origin xyz=-0.215 0.1775 0.06

Commit message: added moving_node

File: agrolab_description/urdf/agrolab.urdf (robot description, URDF)
Before this commit: robot agrolab, 11 links, 10 joints
Joints:
- joint Camera2Light: origin xyz=-0.26 -0.26 0.4 rpy=0 1.57 0 -> xyz=-0.28 -0.26 0.30 rpy=0 1.57079632679 0

Commit message: fixed camera rotation added model for gripper to mesh folder

File: agrolab_description/urdf/agrolab.urdf (robot description, URDF)
Before this commit: robot agrolab, 11 links, 10 joints
Joints:
- joint Camera2Light: axis (none) -> 0 0 -1; limit (none) -> lower=0 upper=0.2 effort=10000 velocity=1; type continuous -> prismatic
- joint gripper: origin xyz=-0.22 -0.26 0.25 rpy=1.57 3.14 0 -> xyz=-0.22 -0.26 0.35 rpy=1.57 3.14 0
- joint gripper_sub: origin xyz=-0.22 -0.26 0.25 rpy=-1.57 0 0 -> xyz=-0.22 -0.26 0.35 rpy=-1.57 0 0

Commit message: added displace by publishing in topic

File: agrolab_description/urdf/agrolab.urdf (robot description, URDF)
Before this commit: robot agrolab, 11 links, 10 joints
Joints:
- joint gripper: origin xyz=-0.22 -0.26 0.35 rpy=1.57 3.14 0 -> xyz=-0.2451 -0.265 0.305 rpy=1.57 3.14 0
- joint gripper_sub: origin xyz=-0.22 -0.26 0.35 rpy=-1.57 0 0 -> xyz=-0.2451 -0.265 0.305 rpy=-1.57 0 0

Commit message: added sphere grasping

File: agrolab_description/urdf/agrolab.urdf (robot description, URDF)
Before this commit: robot agrolab, 11 links, 10 joints
Links:
- removed link sphere1
Joints:
- removed joint sphere1
- joint gripper: origin xyz=-0.2451 -0.265 0.305 rpy=1.57 3.14 0 -> xyz=-0.2451 -0.265 0.260 rpy=1.57 3.14 0
- joint gripper_sub: origin xyz=-0.2451 -0.265 0.305 rpy=-1.57 0 0 -> xyz=-0.2451 -0.265 0.260 rpy=-1.57 0 0
